File: VT100/Hardware/AdapterBoard/VT100-V22/VT100-V22.kicad_pcb (KiCad board)
At the start: 2 copper layers, 99.7 x 99.6 mm, 42 parts, among them J1 GPIO, J2 RS232, J3 Vin < 12V DC / AC, J4 Mini-DIN-6, J5 zu Pi Zero, J6 USB_A, J7 Z80-MBC2 direct, J8 LCD Power, J9 On / Off, K1 G5V-2, Q2 BC546, Q3 BS170, U1 LM2576HVS-ADJ

Commit message: VT100: checkpoint full workspace artifacts
- capture the current VT100 workspace state including generated artifacts
- record the latest local Circle submodule checkpoint
- include rollback release artifacts for targeted recovery
Parts:
- removed R11: 820, Resistor_THT:R_Axial_DIN0207_L6.3mm_D2.5mm_P10.16mm_Horizontal
- removed R12: 1.5k, Resistor_THT:R_Axial_DIN0207_L6.3mm_D2.5mm_P10.16mm_Horizontal
- R2: value 820 -> 1k
- R3: value 1.5k -> 1k
- moved R2 37.5 mm to (156.9, 103.2)
- moved R3 28.0 mm to (156.9, 107.5), turned to 180 degrees
Connections:
- J2 pad 1: +3V3 -> +5V
- J4 pad 3: Net-(J7-Pin_3) -> Net-(J2-Pin_2)
- J4 pad 4: Net-(J7-Pin_4) -> Net-(J2-Pin_3)
- J7 pad 3: Net-(J7-Pin_3) -> Net-(J2-Pin_2)
- J7 pad 4: Net-(J7-Pin_4) -> Net-(J2-Pin_3)
- K1 pad 13: /GPIO15/RXD0 -> Net-(K1-Pad13)
- K1 pad 4: /GPIO14/TXD0 -> Net-(K1-Pad4)
- R2 pad 1: Net-(J2-Pin_3) -> Net-(K1-Pad13)
- R2 pad 2: Net-(J7-Pin_4) -> /GPIO15/RXD0
- R3 pad 1: GND -> Net-(K1-Pad4)
- R3 pad 2: Net-(J2-Pin_3) -> /GPIO14/TXD0
Routing:
- net Net-(J7-Pin_3): track 61.4 -> 0.00 mm
- net +3V3: track 57.7 -> 0.00 mm
- net Net-(J7-Pin_4): track 47.6 -> 0.00 mm
- net +5V: track 240.2 -> 278.8 mm
- net Net-(J2-Pin_2): track 77.3 -> 112.8 mm
- net /GPIO15/RXD0: track 48.7 -> 15.0 mm
- net Net-(J2-Pin_3): track 82.6 -> 115.5 mm
- net Net-(K1-Pad13): track 0.00 -> 23.5 mm
- net /GPIO14/TXD0: track 39.5 -> 19.2 mm
- net Net-(K1-Pad4): track 0.00 -> 10.2 mm
Other:
- board text added: "PI VT100 Adapter Board Version 2.3 4/2026 © R. Zühlsdorff"
- board text removed: "PI VT100 Adapter Board Version 2.2 1/2026 © R. Zühlsdorff"
