File: VT100/Hardware/AdapterBoard/VT100-backups/VT100-2026-01-10_204449 2/PiZero_VT100.kicad_sch (KiCad schematic)
At the start: 42 parts, among them J1 GPIO, J2 RS232, J3 Vin < 12V DC / AC, J4 Mini-DIN-6, J5 zu Pi Zero, J6 USB_A, J7 Z80-MBC2 direct, J8 LCD Power, J9 On / Off, K1 G5V-2, Q2 BC546, Q3 BS170, U1 LM2576HVS-ADJ

Commit message: VT100: checkpoint full workspace artifacts
- capture the current VT100 workspace state including generated artifacts
- record the latest local Circle submodule checkpoint
- include rollback release artifacts for targeted recovery
Parts:
- removed R11: 820, Resistor_THT:R_Axial_DIN0207_L6.3mm_D2.5mm_P10.16mm_Horizontal, symbol Device:R
- removed R12: 1.5k, Resistor_THT:R_Axial_DIN0207_L6.3mm_D2.5mm_P10.16mm_Horizontal, symbol Device:R
Connections:
- net +3V3: no longer J2.1 (Pin_1)
- net +5V: now also J2.1 (Pin_1)
- net GPIO15/RXD0: now also R2.1, R3.2; no longer K1.13
- net at J2.2 (Pin_2), K1.6, K1.9: now also J4.3, J7.3 (Pin_3)
- net at J2.3 (Pin_3), K1.11, K1.8: now also J4.4, J7.4 (Pin_4); no longer R2.1, R3.2
- new net: K1.13, R2.2
Other:
- note added: "MAX232 mit DB9 Stecker auf PCB"
- note added: "Version 2.1 (Fehlerbehebungen) - 40V 2A DIP Gleichrichter verwenden - Hinweise auf Verwendung von LM2576-5.0 statt LM2576-adj - Pads bei SMD Widerständen anpassen für 1206 und 0805"
- note removed: "Level shifted to 3.3V"
- note removed: "MAX3232 mit DB9 Stecker auf PCB"
- note removed: "Version 2.2 (Fehlerbehebungen) - 40V 2A DIP Gleichrichter verwenden - Hinweise auf Verwendung von LM2576-5.0 statt LM2576-adj - Pads bei SMD Widerständen anpassen für 1206 und 0805 - MAX3232 verwenden für 3.3V Kompatibilität - RX Level Shifter mit R2 u. R3 nur für DIN6"
- moved on the sheet: R2, R3
