File: VT100/Hardware/AdapterBoard/VT100-V23/VT100-V23.kicad_pcb (KiCad board)
At the start: 2 copper layers, 99.7 x 99.6 mm, 44 parts, among them J1 GPIO, J2 RS232, J3 Vin < 12V DC / AC, J4 Mini-DIN-6, J5 zu Pi Zero, J6 USB_A, J7 Z80-MBC2 direct, J8 LCD Power, J9 On / Off, K1 G5V-2, Q1 BSS138, Q2 BC546, Q4 BSS138, Q5 BSS138, U1 LM2576HVS-ADJ

Commit message: VT100: add GPIO7-controlled SBC power
Add persistent SBC power configuration and apply it at startup and after modern setup save. Update the V2.3 hardware design and documentation. Firmware build passed; setup behavior was verified, physical hardware validation remains pending.
Parts:
- added Q3: IRL540, Package_TO_SOT_THT:TO-220-3_Vertical, F.Cu at (154.3, 132.8)
- added R13: 100, Resistor_SMD:R_0805_2012Metric_Pad1.20x1.40mm_HandSolder, F.Cu at (163.4, 134.9)
- added R14: 10k, Resistor_SMD:R_0805_2012Metric_Pad1.20x1.40mm_HandSolder, F.Cu at (163.5, 138.0)
- J6: footprint Connector_USB:USB_A_Stewart_SS-52100-001_Horizontal -> Connector_USB:USB_A_Molex_67643_Horizontal
Connections:
- J1 pad 26: /GPIO7/SPI0.CE1 -> SBC ON/OFF
- J1 pad 28: /ID_SCL -> unconnected-(J1-Pin_28-Pad28)
- J4 pad 1: GND -> Net-(J7-Pin_1)
- J4 pad 2: GND -> Net-(J7-Pin_1)
- J4 pad 5: GND -> Net-(J7-Pin_1)
- J7 pad 1: GND -> Net-(J7-Pin_1)
Routing:
- net Net-(J7-Pin_1): track 0.00 -> 55.6 mm
- net SBC ON/OFF: track 0.00 -> 45.4 mm, vias 0 -> 1
- net Net-(Q3-G): track 0.00 -> 9.01 mm
- net Net-(J2-Pin_2): track 95.5 -> 99.3 mm
- net Net-(D3-K): track 62.0 -> 65.6 mm
- net Sound: vias 2 -> 1
Other:
- outline, holes or cut-outs redrawn
- board text added: "PI VT100 Adapter Board Version 2.3 9/2026 © R. Zühlsdorff"
- board text removed: "PI VT100 Adapter Board Version 2.3 4/2026 © R. Zühlsdorff"
