File: VT100/Hardware/AdapterBoard/VT100-V23/VT100-V23.kicad_sch (KiCad schematic)
At the start: 44 parts, among them J1 GPIO, J2 RS232, J3 Vin < 12V DC / AC, J4 Mini-DIN-6, J5 zu Pi Zero, J6 USB_A, J7 Z80-MBC2 direct, J8 LCD Power, J9 On / Off, K1 G5V-2, Q1 BSS138, Q2 BC546, Q4 BSS138, Q5 BSS138, U1 LM2576HVS-ADJ

Commit message: VT100: add GPIO7-controlled SBC power
Add persistent SBC power configuration and apply it at startup and after modern setup save. Update the V2.3 hardware design and documentation. Firmware build passed; setup behavior was verified, physical hardware validation remains pending.
Parts:
- added Q3: IRL540, Package_TO_SOT_THT:TO-220-3_Vertical, symbol Transistor_FET:Q_NMOS_GDS
- added R13: 100, Resistor_SMD:R_0805_2012Metric_Pad1.20x1.40mm_HandSolder, symbol Device:R
- added R14: 10k, Resistor_SMD:R_0805_2012Metric_Pad1.20x1.40mm_HandSolder, symbol Device:R
- J6: footprint Connector_USB:USB_A_Stewart_SS-52100-001_Horizontal -> Connector_USB:USB_A_Molex_67643_Horizontal
Connections:
- net GND: now also Q3.3 (S), R14.1; no longer J4.1, J4.2, J4.5, J6.5 (Shield), J7.1 (Pin_1)
- net GPIO7/SPI0.CE1: no longer J1.26 (Pin_26)
- net ID_SCL: no longer J1.28 (Pin_28)
- new net: Q3.1 (G), R13.2
- new net: J4.1, J4.2, J4.5, J7.1 (Pin_1), Q3.2 (D)
- new net SBC ON/OFF: J1.26 (Pin_26), R13.1, R14.2
- no-connect marks 31 -> 30
Other:
- note added: "Optional: Wenn Schnittstelle permanent an 5V liegen soll einfach 2 und 3 brücken!"
- note added: "SBC Power On Switch"
- note added: "Version 2.3 (Fehlerbehebungen) - 40V 2A DIP Gleichrichter verwenden - Hinweise auf Verwendung von LM2576-5.0 statt LM2576-adj - Pads bei SMD Widerständen anpassen für 1206 und 0805 - RX / TX Level Shifter mit PMOS BSS138 für echte 3,3V/5V Umsetzung - 5V der SBC Schnittstelle kann über Pi GPIO7 geschaltet werden - USB-A auf Top Mount Variante MOLEX 67643 umgestellt"
- note removed: "Version 2.3 (Fehlerbehebungen) - 40V 2A DIP Gleichrichter verwenden - Hinweise auf Verwendung von LM2576-5.0 statt LM2576-adj - Pads bei SMD Widerständen anpassen für 1206 und 0805 - RX / TX Level Shifter mit PMOS BSS138 für ecte 3,3V/5V Umsetzung"
- note removed: "echten lavel Shufter 3.3V nach 5V"
- moved on the sheet: J4
